File: RTL8720DN multi function board/RTL8720DN multi function board.kicad_pcb (KiCad board)
At the start: 2 copper layers, 55 x 28 mm, 25 parts, among them J1 Mag Switch, J2 UART, J3 Power, J4 GPIO2, J5 GPIO1, J6 GPIO3, SW1 RESET, SW2 DNLOAD, U1 BW16, U2 74HC02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

Commit message: pcb and rtlduino update
Parts:
- added J7: Pwr, Connector_PinHeader_2.54mm:PinHeader_1x02_P2.54mm_Vertical, F.Cu at (159.5, 107.7)
- added J8: Pwr, Connector_PinHeader_2.54mm:PinHeader_1x01_P2.54mm_Vertical, F.Cu at (162.1, 95.0)
- moved SW1 0.51 mm to (165.6, 104.1)
Routing:
- net +3V3: track 48.3 -> 59.0 mm
- net Net-(C3-Pad1): track 24.8 -> 32.7 mm
- net GND: track 99.0 -> 103.3 mm
Other:
- board text added: "3.3V_OUT"
- board text added: "5V_OUT"

Commit message: Documentation Corrections
Other:
- board text added: "PB3"
- board text removed: "PA3"
Changed lines of the file:
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@@
   )
   (setup
-    (last_trace_width 0.5)
+    (last_trace_width 0.25)
     (user_trace_width 0.4)
     (user_trace_width 0.5)
@@
   (gr_line (start 115.4 90.42) (end 120.55 90.42) (layer Edge.Cuts) (width 0.12))
   (gr_line (start 115.4 108.712) (end 115.4 113.885) (layer Edge.Cuts) (width 0.12))
-  (gr_text PA3 (at 124.968 113.284) (layer F.SilkS)
+  (gr_text PB3 (at 124.968 113.284) (layer F.SilkS)
     (effects (font (size 0.6 0.6) (thickness 0.15)))
   )
